Commit message: COD: 接入 URDF + 默认配置；Kp40/Kd2

File: plane/resources/robots/cod_V1/urdf/COD_2026_Balance_3_0.urdf (robot description, URDF)
Before this commit: robot COD-2026-Balance-2.0, 15 links, 14 joints
Joints:
- joint Left_front_joint: origin xyz=-0.01939139612421 -0.183700000000001 -0.0500000000000005 rpy=0 0 0 -> xyz=0 -0.0240 0 rpy=0 0 0; parent base_link -> Left_rear_link
- joint Right_front_joint: origin xyz=-0.01939139612421 0.181699999999995 -0.0500000000000005 rpy=0 0 0 -> xyz=0 +0.0240 0 rpy=0 0 0; parent base_link -> Right_rear_link
